Commit message: edit aruco_marker_link orientation, autonomous navigation now works

File: install/boxing_bot_description/share/boxing_bot_description/src/description/boxing_bot_description.urdf (robot description, URDF)
Before this commit: robot boxing_bot, 4 links, 3 joints
Joints:
- joint base_to_aruco_marker: origin xyz=0 0 ${(base_height/2) + 0.0005} rpy=0 0 0 -> xyz=0 0 ${(base_height/4) + 0.0005} rpy=0 0 -1.5709

Commit message: more realistic URDF, changed castwheel to box shape to reduce jerky motion in simulation

File: install/boxing_bot_description/share/boxing_bot_description/src/description/boxing_bot_description.urdf (robot description, URDF)
Before this commit: robot boxing_bot, 4 links, 3 joints
Links:
- added link back_caster; collision box size=${wheel_radius} ${wheel_radius} ${wheel_radius}; visual box size=${wheel_radius} ${wheel_radius} ${wheel_radius}
- added link upper_body; collision cylinder length=${upper_body_height} radius=${base_radius}; visual cylinder length=${upper_body_height} radius=${base_radius}
- link base_link: geometry collision cylinder length=${base_height} radius=${base_radius}; visual cylinder length=${base_height} radius=${base_radius}
- link front_caster: geometry collision box size=${wheel_radius} ${wheel_radius} ${wheel_radius}; visual box size=${wheel_radius} ${wheel_radius} ${wheel_radius}
Joints:
- removed joint caster_joint
- added joint back_caster_joint: type fixed, parent base_link, child back_caster, origin xyz=${-(caster_xoff)} 0.0 ${-(base_height/2) + 0.001} rpy=0 0 0
- added joint front_caster_joint: type fixed, parent base_link, child front_caster, origin xyz=${(caster_xoff)} 0.0 ${-(base_height/2) + 0.001} rpy=0 0 0
- added joint upper_body_joint: type fixed, parent base_link, child upper_body, origin xyz=0.0 0.0 ${(base_height)*2 + (wheel_radius)} rpy=0 0 0
- joint base_to_aruco_marker: origin xyz=0 0 ${(base_height/4) + 0.0005} rpy=0 0 -1.5709 -> xyz=0 0 ${(base_height)/2 +(upper_body_height)} rpy=0 0 -1.5709

File: install/boxing_bot_description/share/boxing_bot_description/src/description/boxing_bot_description_orig.urdf (robot description, URDF)
Before this commit: robot boxing_bot, 4 links, 3 joints
Joints:
- joint base_to_aruco_marker: origin xyz=0 0 ${-(base_height/4) - 0.0005} rpy=0 0 0 -> xyz=0 0 ${(base_height/4) + 0.0005} rpy=0 0 -1.5709

Commit message: multiple aruco markers detection and EKF, boxing bot  URDF updated

File: install/boxing_bot_description/share/boxing_bot_description/src/description/boxing_bot_description.urdf (robot description, URDF)
Before this commit: robot boxing_bot, 6 links, 5 joints
Links:
- removed link aruco_marker_link
- added link aruco_marker_0_link; collision box size=0.09 0.09 0.001; visual box size=0.09 0.09 0.001
- added link aruco_marker_1_link; collision box size=0.09 0.09 0.001; visual box size=0.09 0.09 0.001
- added link aruco_marker_2_link; collision box size=0.09 0.09 0.001; visual box size=0.09 0.09 0.001
- added link aruco_marker_3_link; collision box size=0.09 0.09 0.001; visual box size=0.09 0.09 0.001
Joints:
- removed joint base_to_aruco_marker
- added joint base_to_aruco_marker_0: type fixed, parent base_link, child aruco_marker_0_link, origin xyz=0.1 0 ${(base_height)/2 +(upper_body_height)} rpy=0 0 -1.5709
- added joint base_to_aruco_marker_1: type fixed, parent base_link, child aruco_marker_1_link, origin xyz=0 0.1 ${(base_height)/2 +(upper_body_height)} rpy=0 0 -1.5709
- added joint base_to_aruco_marker_2: type fixed, parent base_link, child aruco_marker_2_link, origin xyz=-0.1 0 ${(base_height)/2 +(upper_body_height)} rpy=0 0 -1.5709
- added joint base_to_aruco_marker_3: type fixed, parent base_link, child aruco_marker_3_link, origin xyz=0 -0.1 ${(base_height)/2 +(upper_body_height)} rpy=0 0 -1.5709

Commit message: some edits to robot_localization

File: install/boxing_bot_description/share/boxing_bot_description/src/description/boxing_bot_description.urdf (robot description, URDF)
Before this commit: robot boxing_bot, 9 links, 8 joints
Links:
- added link strike_bar; collision cylinder length=0.5 radius=0.05; visual cylinder length=0.5 radius=0.05
Joints:
- added joint strike_bar_joint: type fixed, parent upper_body, child strike_bar, origin xyz=0.0 0.0 ${(upper_body_height)/2 + 0.25} rpy=0 0 0
